Commit message: save

File: src/system/roombot_gazebo/xacro/roomba_stl_body.xacro (robot description, xacro)
@@ -5,4 +5,7 @@
   <material name="grey">
     <color rgba="0.5 0.5 0.5 2.5"/>
+  </material>
+  <material name="blue">
+    <color rgba="0.0 0.0 1.0 2.5"/>
   </material>
   <xacro:macro name="wheel_macro" params="parent prefix xyz">
@@ -109,4 +112,59 @@
     <mu2 value="0.5" />
   </gazebo>
+  <xacro:macro name="laser_macro" params="parent prefix xyz">
+    <joint name="${prefix}_joint" type="fixed">
+      <parent link="${parent}"/>
+      <child  link="${prefix}_link"/>
+      <origin xyz="${xyz}" rpy="0 0 0"/>
+    </joint>
+    <link name="${prefix}_link">
+      <visual>
+        <origin xyz="0 0 0" rpy="0 0 0" />
+        <geometry>
+          <cylinder radius="0.02" length="0.06" />
+        </geometry>
+        <material name="blue" />
+      </visual>
+      <collision>
+        <origin xyz="0 0 0" rpy="0 0 0"/>
+        <geometry>
+          <cylinder radius="0.02" length="0.06" />
+        </geometry>
+      </collision>
+    </link>
+    <gazebo reference="${prefix}_link">
+      <material>Gazebo/Blue</material>
+      <sensor type="ray" name="${prefix}">
+        <pose>0 0 0 0 0 0</pose>
+        <visualize>false</visualize>
+        <update_rate>10</update_rate>
+        <ray>
+          <scan>
+            <horizontal>
+              <samples>400</samples>
+              <resolution>1</resolution>
+              <min_angle>${radians(-90)}</min_angle>
+              <max_angle>${radians( 90)}</max_angle>
+            </horizontal>
+          </scan>
+          <range>
+            <min>0.10</min>
+            <max>20.0</max>
+            <resolution>0.01</resolution>
+          </range>
+          <noise>
+            <type>gaussian</type>
+            <mean>0.0</mean>
+            <stddev>0.01</stddev>
+          </noise>
+        </ray>
+        <plugin name="gazebo_ros_lidar_controller" filename="libgazebo_ros_laser.so">
+          <topicName>/${prefix}_link/scan</topicName>
+          <frameName>${prefix}_link</frameName>
+        </plugin>
+      </sensor>
+    </gazebo>
+  </xacro:macro>
+  <xacro:laser_macro prefix="lidar" parent="base_link" xyz="-0.05 0 0.14"/>
   <xacro:macro name="imu_macro" params="parent prefix xyz">
     <joint name="imu_joint" type="fixed">
